File: YonderDeep/YonderDeep.kicad_sch (KiCad schematic)
At the start: 16 parts, among them J1 GPIO, U1 CAT24C256

Commit message: Working on PCB placement
Parts:
- 5V_in1: renamed from 5V_in; footprint (none) -> TerminalBlock_MetzConnect:TerminalBlock_MetzConnect_Type701_RT11L02HGLU_1x02_P6.35mm_Horizontal
- BACK1: renamed from BACK; footprint (none) -> Capacitor_THT:C_Rect_L7.0mm_W2.5mm_P5.00mm
- FRONT1: renamed from FRONT; footprint (none) -> Capacitor_THT:C_Rect_L7.0mm_W2.5mm_P5.00mm
- J2: renamed from J?; footprint (none) -> LED_THT:LED_D3.0mm
- JPressure_Sensor_Breakout_Right1: renamed from JPressure_Sensor_Breakout_Right; footprint (none) -> Connector_PinHeader_2.54mm:PinHeader_1x04_P2.54mm_Vertical
- LEFT1: renamed from LEFT; footprint (none) -> Capacitor_THT:C_Rect_L7.0mm_W2.5mm_P5.00mm
- Pressure_Sensor_Breakout_Left1: renamed from Pressure_Sensor_Breakout_Left; footprint (none) -> Connector_PinHeader_2.54mm:PinHeader_1x04_P2.54mm_Vertical
- RIGHT1: renamed from RIGHT; footprint (none) -> Capacitor_THT:C_Rect_L7.0mm_W2.5mm_P5.00mm
Connections:
- net GPIO[18]/PCM.CLK is gone; now on net Back_Motor: J1.12 (Pin_12)
- net GPIO[24] is gone; now on net Front_Motor: J1.18 (Pin_18)
- net GPIO[4]/GPCLK0 is gone; now on net GND: J1.7 (Pin_7)
- net GND: now also LEFT1.1 (Pin_1)
- net Back_Motor: now reaches BACK1.1 (Pin_1)
- net Front_Motor: now reaches FRONT1.1 (Pin_1)
