File: YonderDeep/_autosave-YonderDeep.kicad_pcb (KiCad board)
At the start: 2 copper layers, 65 x 56 mm, 18 parts, among them J1 GPIO

Commit message: DRC no error
Connections:
- J1 pad 1: 3.3V -> unconnected-(J1-Pad1)
Routing:
- net GND: track 258.9 -> 0.00 mm
- net Front_Motor: track 87.7 -> 0.00 mm
- net /GPIO[6]: track 77.5 -> 0.00 mm
- net Right_Motor: track 0.00 -> 54.2 mm, vias 0 -> 1
- net Back_Motor: track 69.3 -> 115.8 mm
- net Left_Motor: track 98.6 -> 58.4 mm
- net IMU_RST: track 0.00 -> 39.1 mm, vias 0 -> 1
- net 3.3V: track 62.6 -> 55.3 mm
- net SDA1: track 80.6 -> 85.2 mm
- net LED_GPIO12: track 13.6 -> 15.6 mm
- net SCL1: track 85.8 -> 84.2 mm
